File: HDK/Dashboard-NumberIndicators.kicad_sch (KiCad schematic)
At the start: 7 parts, among them J101 Conn_02x08_Odd_Even, U101 CA56-12EWA, U102 CA56-12EWA

Commit message: updated bom
Parts:
- removed H101, H102, H103, H104: MountingHole_Pad, MountingHole:MountingHole_3.2mm_M3_DIN965_Pad_TopBottom, symbol Mechanical:MountingHole_Pad
- removed J101: Conn_02x08_Odd_Even, Connector_JST:JST_PHD_B16B-PHDSS_2x08_P2.00mm_Vertical, symbol Connector_Generic:Conn_02x08_Odd_Even
- removed U101, U102: CA56-12EWA, Display_7Segment:CA56-12EWA, symbol Display_Character:CA56-12EWA
Other:
- note removed: "7 Segment Display Arrays"
- note removed: "DB->DB-NI"
